File: Sofle_Cho_Extra_Stagger/PCB/SofleKeyboard.kicad_pcb (KiCad board)
At the start: 2 copper layers, 159.3 x 123.4 mm, 84 parts, among them J2 4PIN, J3 OLED, P1 i2c_pin, P2 i2c_pin, SW1 SW_PUSH_LED, SW10 SW_PUSH_LED, SW11 SW_PUSH_LED, SW12 SW_PUSH_LED, SW13 SW_PUSH_LED, SW14 SW_PUSH_LED, SW15 SW_PUSH_LED, SW16 SW_PUSH_LED, SW17 SW_PUSH_LED, SW18 SW_PUSH_LED, SW19 SW_PUSH_LED, SW2 SW_PUSH_LED, SW20 SW_PUSH_LED, SW21 SW_PUSH_LED, SW22 SW_PUSH_LED, SW23 SW_PUSH_LED, SW24 SW_PUSH_LED, SW25 Rotary_Encoder_Switch, SW26 SW_PUSH_LED, SW27 SW_PUSH_LED, SW28 SW_PUSH_LED, SW29 SW_PUSH_LED, SW3 SW_PUSH_LED, SW30 SW_PUSH_LED, SW4 SW_PUSH_LED, SW5 SW_PUSH_LED, SW6 SW_PUSH_LED, SW7 SW_PUSH_LED, SW8 SW_PUSH_LED, SW9 SW_PUSH_LED, U1 ProMicro

Commit message: Change PCB layout, fairly good new 'good enough' point
Routing:
- net col1: track 333.4 -> 327.2 mm
- net col0: track 341.5 -> 335.8 mm
- net VCC: track 922.2 -> 919.2 mm
- net col2: track 311.2 -> 308.4 mm
- net row3: track 175.0 -> 172.4 mm
- net Net-(SW4-Pad2): track 56.2 -> 54.4 mm
- net row2: track 156.1 -> 157.8 mm, vias 7 -> 8
- net GND: track 1119.2 -> 1118.3 mm
- net Net-(SW29-Pad2): track 46.8 -> 47.4 mm
- net row0: track 154.7 -> 155.2 mm
Other:
- board size 159.3 x 123.4 mm -> 143.4 x 114.2 mm
- board text added: "Sofle Choc Extra Stagger v1.0 by Flippie van Dyk"
- board text removed: "Sofle Choc v2.1 by Brian Low"
